File: Circuit/boneIO - relay board 32x5A/boneIO - relay board 32x5A.sch (KiCad schematic (older format))
At the start: 80 parts, among them J1 Screw_Terminal_01x03, J10 Screw_Terminal_01x03, J11 Screw_Terminal_01x03, J12 Conn_02x04_Odd_Even, J13 Screw_Terminal_01x03, J14 Screw_Terminal_01x03, J15 Screw_Terminal_01x03, J16 Screw_Terminal_01x03, J17 Screw_Terminal_01x03, J2 Screw_Terminal_01x03, J3 Screw_Terminal_01x03, J4 Screw_Terminal_01x03, J5 Screw_Terminal_01x03, J6 Screw_Terminal_01x03, J7 Screw_Terminal_01x03, J8 Screw_Terminal_01x03, J9 Screw_Terminal_01x03, K1 HF46F, K10 HF46F, K11 HF46F, K12 HF46F, K13 HF46F, K14 HF46F, K15 HF46F, K16 HF46F, K17 HF46F, K18 HF46F, K19 HF46F, K2 HF46F, K20 HF46F, K21 HF46F, K22 HF46F, K23 HF46F, K24 HF46F, K25 HF46F, K26 HF46F, K27 HF46F, K28 HF46F, K29 HF46F, K3 HF46F, K30 HF46F, K31 HF46F, K32 HF46F, K4 HF46F, K5 HF46F, K6 HF46F, K7 HF46F, K8 HF46F, K9 HF46F, SW1 SW_DIP_x03, SW2 SW_DIP_x03, SW3 SW_DIP_x03, U1 MCP23017_SS, U2 ULN2803A, U3 ULN2803A, U4 MCP23017_SS, U5 ULN2803A, U6 ULN2803A, U7 MCP9808_MSOP

Commit message: relay 32x5 directory cleanup
added shared library with footprints
Parts:
- J12: footprint ph80ds-21:PinHeader_2x04_P2.54mm_Vertical -> boneIO:PinHeader_2x04_P2.54mm_Vertical
- K1, K10, K11, K12, K13, K14, K15, K16, K17, K18, K19, K2, K20, K21, K22, K23, K24, K25, K26, K27, K28, K29, K3, K30, K31, K32, K4, K5, K6, K7, K8, K9: footprint HF46F:HF46F -> boneIO:HF46F; symbol HF46F:HF46F -> boneIO:HF46F
- U7: symbol Sensor_Temperature:MCP9808_MSOP -> boneIO:MCP9808_MSOP
