File: Circuit/boneIO - relay board 32x5A/boneIO - relay board 32x5A.sch (KiCad schematic (older format))
At the start: 80 parts, among them J1 Screw_Terminal_01x03, J10 Screw_Terminal_01x03, J11 Screw_Terminal_01x03, J12 Conn_02x04_Odd_Even, J13 Screw_Terminal_01x03, J14 Screw_Terminal_01x03, J15 Screw_Terminal_01x03, J16 Screw_Terminal_01x03, J17 Screw_Terminal_01x03, J2 Screw_Terminal_01x03, J3 Screw_Terminal_01x03, J4 Screw_Terminal_01x03, J5 Screw_Terminal_01x03, J6 Screw_Terminal_01x03, J7 Screw_Terminal_01x03, J8 Screw_Terminal_01x03, J9 Screw_Terminal_01x03, K1 HF46F, K10 HF46F, K11 HF46F, K12 HF46F, K13 HF46F, K14 HF46F, K15 HF46F, K16 HF46F, K17 HF46F, K18 HF46F, K19 HF46F, K2 HF46F, K20 HF46F, K21 HF46F, K22 HF46F, K23 HF46F, K24 HF46F, K25 HF46F, K26 HF46F, K27 HF46F, K28 HF46F, K29 HF46F, K3 HF46F, K30 HF46F, K31 HF46F, K32 HF46F, K4 HF46F, K5 HF46F, K6 HF46F, K7 HF46F, K8 HF46F, K9 HF46F, SW1 SW_DIP_x03, SW2 SW_DIP_x03, SW3 SW_DIP_x03, U1 MCP23017_SS, U2 ULN2803A, U3 ULN2803A, U4 MCP23017_SS, U5 ULN2803A, U6 ULN2803A, U7 MCP9808_MSOP

Commit message: Merge Kamil's changes
Parts:
- K1, K10, K11, K12, K13, K14, K15, K16, K17, K18, K19, K2, K20, K21, K22, K23, K24, K25, K26, K27, K28, K29, K3, K30, K31, K32, K4, K5, K6, K7, K8, K9: symbol boneIO:HF46F -> boneIO---relay-board-32x5A-rescue:HF46F-boneIO
- U7: symbol boneIO:MCP9808_MSOP -> boneIO---relay-board-32x5A-rescue:MCP9808_MSOP-boneIO
Changed lines of the file:
@@
 	17625 2625 17625 2725
 $Comp
-L boneIO:MCP9808_MSOP U7
+L boneIO---relay-board-32x5A-rescue:MCP9808_MSOP-boneIO U7
 U 1 1 61B8C06C
 P 21000 2925
@@
 	20550 3025 20600 3025
 $Comp
-L boneIO:HF46F K1
+L boneIO---relay-board-32x5A-rescue:HF46F-boneIO K1
 U 1 1 61B88957
 P 3400 7800
@@
 $EndComp
 $Comp
-L boneIO:HF46F K2
+L boneIO---relay-board-32x5A-rescue:HF46F-boneIO K2
 U 1 1 61B8A916
 P 3400 8850
@@
 $EndComp
 $Comp
-L boneIO:HF46F K3
+L boneIO---relay-board-32x5A-rescue:HF46F-boneIO K3
 U 1 1 62B1A65F
 P 3400 10150
@@
 $EndComp
 $Comp
-L boneIO:HF46F K4
+L boneIO---relay-board-32x5A-rescue:HF46F-boneIO K4
 U 1 1 62B1A668
 P 3400 11200
@@
 $EndComp
 $Comp
-L boneIO:HF46F K5
+L boneIO---relay-board-32x5A-rescue:HF46F-boneIO K5
 U 1 1 62B2A576
 P 3400 12500
@@
 $EndComp
 $Comp
-L boneIO:HF46F K6
+L boneIO---relay-board-32x5A-rescue:HF46F-boneIO K6
 U 1 1 62B2A57F
 P 3400 13550
@@
 $EndComp
 $Comp
-L boneIO:HF46F K7
+L boneIO---relay-board-32x5A-rescue:HF46F-boneIO K7
 U 1 1 62C5A60C
 P 7000 7800
@@
 $EndComp
 $Comp
-L boneIO:HF46F K8
+L boneIO---relay-board-32x5A-rescue:HF46F-boneIO K8
 U 1 1 62C5A615
 P 7000 8850
@@
 $EndComp
 $Comp
-L boneIO:HF46F K9
+L boneIO---relay-board-32x5A-rescue:HF46F-boneIO K9
 U 1 1 62C5A63D
 P 7000 10150
@@
 $EndComp
 $Comp
-L boneIO:HF46F K10
+L boneIO---relay-board-32x5A-rescue:HF46F-boneIO K10
 U 1 1 62C5A646
 P 7000 11200
@@
 $EndComp
 $Comp
-L boneIO:HF46F K11
+L boneIO---relay-board-32x5A-rescue:HF46F-boneIO K11
 U 1 1 62C5A66C
 P 7000 12500
@@
 $EndComp
 $Comp
-L boneIO:HF46F K12
+L boneIO---relay-board-32x5A-rescue:HF46F-boneIO K12
 U 1 1 62C5A675
 P 7000 13550
@@
 $EndComp
 $Comp
-L boneIO:HF46F K13
+L boneIO---relay-board-32x5A-rescue:HF46F-boneIO K13
 U 1 1 62C73758
 P 10750 7800
@@
 $EndComp
 $Comp
-L boneIO:HF46F K14
+L boneIO---relay-board-32x5A-rescue:HF46F-boneIO K14
 U 1 1 62C73761
 P 10750 8850
@@
 $EndComp
 $Comp
-L boneIO:HF46F K15
+L boneIO---relay-board-32x5A-rescue:HF46F-boneIO K15
 U 1 1 62C73789
 P 10750 10150
@@
 $EndComp
 $Comp
-L boneIO:HF46F K16
+L boneIO---relay-board-32x5A-rescue:HF46F-boneIO K16
 U 1 1 62C73792
 P 10750 11200
@@
 	10250 11400 10750 11400
 $Comp
-L boneIO:HF46F K17
+L boneIO---relay-board-32x5A-rescue:HF46F-boneIO K17
 U 1 1 62CC3428
 P 14100 7800
@@
 $EndComp
 $Comp
-L boneIO:HF46F K18
+L boneIO---relay-board-32x5A-rescue:HF46F-boneIO K18
 U 1 1 62CC3431
 P 14100 8850
@@
 	14600 7600 14100 7600
 $Comp
-L boneIO:HF46F K19
+L boneIO---relay-board-32x5A-rescue:HF46F-boneIO K19
 U 1 1 6326F0BD
 P 14100 10150
@@
 $EndComp
 $Comp
-L boneIO:HF46F K20
+L boneIO---relay-board-32x5A-rescue:HF46F-boneIO K20
 U 1 1 6326F0C6
 P 14100 11200
@@
 	14600 9950 14100 9950
 $Comp
-L boneIO:HF46F K21
+L boneIO---relay-board-32x5A-rescue:HF46F-boneIO K21
 U 1 1 6328F764
 P 14100 12650
@@
 $EndComp
 $Comp
-L boneIO:HF46F K22
+L boneIO---relay-board-32x5A-rescue:HF46F-boneIO K22
 U 1 1 6328F76D
 P 14100 13700
@@
 	14600 12450 14100 12450
 $Comp
-L boneIO:HF46F K23
+L boneIO---relay-board-32x5A-rescue:HF46F-boneIO K23
 U 1 1 632BAFD0
 P 17550 7750
@@
 $EndComp
 $Comp
-L boneIO:HF46F K24
+L boneIO---relay-board-32x5A-rescue:HF46F-boneIO K24
 U 1 1 632BAFD9
 P 17550 8800
@@
 	18050 7550 17550 7550
 $Comp
-L boneIO:HF46F K25
+L boneIO---relay-board-32x5A-rescue:HF46F-boneIO K25
 U 1 1 632BAFFF
 P 17550 10100
@@
 $EndComp
 $Comp
-L boneIO:HF46F K26
+L boneIO---relay-board-32x5A-rescue:HF46F-boneIO K26
 U 1 1 632BB008
 P 17550 11150
@@
 	18050 9900 17550 9900
 $Comp
-L boneIO:HF46F K27
+L boneIO---relay-board-32x5A-rescue:HF46F-boneIO K27
 U 1 1 632BB02E
 P 17550 12600
@@
 $EndComp
 $Comp
-L boneIO:HF46F K28
+L boneIO---relay-board-32x5A-rescue:HF46F-boneIO K28
 U 1 1 632BB037
 P 17550 13650
@@
 	18050 12400 17550 12400
 $Comp
-L boneIO:HF46F K29
+L boneIO---relay-board-32x5A-rescue:HF46F-boneIO K29
 U 1 1 632EF485
 P 20750 7750
@@
 $EndComp
 $Comp
-L boneIO:HF46F K30
+L boneIO---relay-board-32x5A-rescue:HF46F-boneIO K30
 U 1 1 632EF48E
 P 20750 8800
@@
 	21250 7550 20750 7550
 $Comp
-L boneIO:HF46F K31
+L boneIO---relay-board-32x5A-rescue:HF46F-boneIO K31
 U 1 1 632EF4B4
 P 20750 10100
@@
 $EndComp
 $Comp
-L boneIO:HF46F K32
+L boneIO---relay-board-32x5A-rescue:HF46F-boneIO K32
 U 1 1 632EF4BD
 P 20750 11150

Commit message: 32x5 v0.3
Parts:
- removed K1, K10, K11, K12, K13, K14, K15, K16, K17, K18, K19, K2, K20, K21, K22, K23, K24, K25, K26, K27, K28, K29, K3, K30, K31, K32, K4, K5, K6, K7, K8, K9: HF46F, boneIO:HF46F, symbol boneIO---relay-board-32x5A-rescue:HF46F-boneIO
- removed R2, R6: 10k, Resistor_SMD:R_0603_1608Metric, symbol Device:R
- removed SW1, SW2, SW3: SW_DIP_x03, Button_Switch_SMD:SW_DIP_SPSTx03_Slide_KingTek_DSHP03TJ_W5.25mm_P1.27mm_JPin, symbol Switch:SW_DIP_x03
- removed U7: MCP9808_MSOP, Package_SO:MSOP-8_3x3mm_P0.65mm, symbol boneIO---relay-board-32x5A-rescue:MCP9808_MSOP-boneIO
- added C7: 100n, Capacitor_SMD:C_0603_1608Metric, symbol Device:C
- added JP1, JP10, JP2, JP3, JP4, JP5, JP6, JP8, JP9: NO_Small, Jumper:SolderJumper-2_P1.3mm_Open_RoundedPad1.0x1.5mm, symbol Device:Jumper_NO_Small
- added K1, K10, K11, K12, K13, K14, K15, K16, K17, K18, K19, K2, K20, K21, K22, K23, K24, K25, K26, K27, K28, K29, K3, K30, K31, K32, K4, K5, K6, K7, K8, K9: HF46F, boneIO_LOGO:HF46F, symbol Relay:UMS05-1A80-75L
- added R15: 4.7k, Resistor_SMD:R_0603_1608Metric, symbol Device:R
- added R4, R8: 10k, Resistor_SMD:R_0603_1608Metric, symbol Device:R
- added U7: MCP9808_SO8, Package_SO:SO-8_3.9x4.9mm_P1.27mm, symbol Sensor_Temperature:MCP9804_MSOP
- added U8: MCP9808_MSOP, Package_SO:MSOP-8_3x3mm_P0.65mm, symbol Sensor_Temperature:MCP9804_MSOP
- J12: footprint boneIO:PinHeader_2x04_P2.54mm_Vertical -> Connector_PinHeader_2.54mm:PinHeader_2x04_P2.54mm_Vertical
- renumbered JP1 to JP7, R4 to R2, R8 to R6
Connections:
- net +3V3: now also C7.1, JP1.1, JP10.1, JP2.1, JP3.1, JP4.1, JP5.1, JP6.1, JP8.1, JP9.1, R15.1, U7.8 (VDD), U8.8 (VDD)
- net GND: now also C7.2, R4.2, R8.2, U7.4 (GND), U8.4 (GND)
- net RELAY1: now also K1.2
- net RELAY10: now also K10.2
- net RELAY11: now also K11.2
- net RELAY12: now also K12.2
- net RELAY13: now also K13.2
- net RELAY14: now also K14.2
- net RELAY15: now also K15.2
- net RELAY16: now also K16.2
- net RELAY17: now also K17.2
- net RELAY18: now also K18.2
- net RELAY19: now also K19.2
- net RELAY2: now also K2.2
- net RELAY20: now also K20.2
- net RELAY21: now also K21.2
- net RELAY22: now also K22.2
- net RELAY23: now also K23.2
- net RELAY24: now also K24.2
- net RELAY25: now also K25.2
- net RELAY26: now also K26.2
- net RELAY27: now also K27.2
- net RELAY28: now also K28.2
- net RELAY29: now also K29.2
- net RELAY3: now also K3.2
- net RELAY30: now also K30.2
- net RELAY31: now also K31.2
- net RELAY32: now also K32.2
- net RELAY4: now also K4.2
- net RELAY5: now also K5.2
- net RELAY6: now also K6.2
- net RELAY7: now also K7.2
- net RELAY8: now also K8.2
- net RELAY9: now also K9.2
- net SCL: now also U7.2 (SCL), U8.2 (SCL)
- net SDA: now also U7.1 (SDA), U8.1 (SDA)
- net VCC: now also K1.1, K10.1, K11.1, K12.1, K13.1, K14.1, K15.1, K16.1, K17.1, K18.1, K19.1, K2.1, K20.1, K21.1, K22.1, K23.1, K24.1, K25.1, K26.1, K27.1, K28.1, K29.1, K3.1, K30.1, K31.1, K32.1, K4.1, K5.1, K6.1, K7.1, K8.1, K9.1
- net at U4.15 (A0): now also JP6.2, R8.1; no longer R5.1
- net at U4.16 (A1): now also R7.1, JP5.2
- net at U4.17 (A2): now also R5.1, JP4.2; no longer R7.1
- net at U1.15 (A0): now also JP3.2, R4.1; no longer R1.1
- net at U1.16 (A1): now also R3.1, JP2.2
- net at U1.17 (A2): now also R1.1, JP1.2; no longer R3.1
- net at R11.1: now also JP8.2, U7.7 (A0), U8.7 (A0)
- net at R12.1: now also JP9.2, U7.6 (A1), U8.6 (A1)
- net at R13.1: now also JP10.2, U7.5 (A2), U8.5 (A2)
- net at J1.1 (Pin_1): now also K1.3, K2.3
- net at J1.2 (Pin_2): now also K1.4
- net at J1.3 (Pin_3): now also K2.4
- net at R14.2: now also U7.3 (Alert)
- net at J2.1 (Pin_1): now also K3.3, K4.3
- net at J2.2 (Pin_2): now also K3.4
- net at J2.3 (Pin_3): now also K4.4
- net at J3.1 (Pin_1): now also K5.3, K6.3
- net at J3.2 (Pin_2): now also K5.4
- net at J3.3 (Pin_3): now also K6.4
- net at J4.1 (Pin_1): now also K7.3, K8.3
- net at J4.2 (Pin_2): now also K7.4
- net at J4.3 (Pin_3): now also K8.4
- net at J5.1 (Pin_1): now also K10.3, K9.3
- net at J5.2 (Pin_2): now also K9.4
- net at J5.3 (Pin_3): now also K10.4
- net at J6.1 (Pin_1): now also K11.3, K12.3
- net at J6.2 (Pin_2): now also K11.4
- net at J6.3 (Pin_3): now also K12.4
- net at J7.1 (Pin_1): now also K13.3, K14.3
- net at J7.2 (Pin_2): now also K13.4
- net at J7.3 (Pin_3): now also K14.4
- net at J8.1 (Pin_1): now also K15.3, K16.3
- net at J8.2 (Pin_2): now also K15.4
- net at J8.3 (Pin_3): now also K16.4
- net at J9.1 (Pin_1): now also K17.3, K18.3
- net at J9.2 (Pin_2): now also K18.4
- net at J9.3 (Pin_3): now also K17.4
- net at J10.1 (Pin_1): now also K19.3, K20.3
- net at J10.3 (Pin_3): now also K19.4
- net at J10.2 (Pin_2): now also K20.4
- net at J11.1 (Pin_1): now also K21.3, K22.3
- net at J11.3 (Pin_3): now also K21.4
- net at J11.2 (Pin_2): now also K22.4
- net at J13.1 (Pin_1): now also K23.3, K24.3
- net at J13.3 (Pin_3): now also K23.4
- net at J13.2 (Pin_2): now also K24.4
- net at J14.1 (Pin_1): now also K25.3, K26.3
- net at J14.3 (Pin_3): now also K25.4
- net at J14.2 (Pin_2): now also K26.4
- net at J15.1 (Pin_1): now also K27.3, K28.3
- net at J15.3 (Pin_3): now also K27.4
- net at J15.2 (Pin_2): now also K28.4
- net at J16.1 (Pin_1): now also K29.3, K30.3
- net at J16.3 (Pin_3): now also K29.4
- net at J16.2 (Pin_2): now also K30.4
- net at J17.1 (Pin_1): now also K31.3, K32.3
- net at J17.3 (Pin_3): now also K31.4
- net at J17.2 (Pin_2): now also K32.4
- new net: R15.2, U8.3 (Alert)
Other:
- note added: "- relay board 32x5A v0.3"
- note added: "ADDRESS\n 0x21"
- note added: "ADDRESS\n 0x48"
- note added: "ADDRESS\n0x20"
- note added: "MCP23017"
- moved on the sheet: C1, C2, C3, C4, C5, C6, J10, J11, J12, J13, J14, J15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
