File: boneIO - relay board 32x5A.kicad_pcb (KiCad board)
At the start: 2 copper layers, 197 x 102 mm, 90 parts, among them J1 Screw_Terminal_01x03, J10 Screw_Terminal_01x03, J11 Screw_Terminal_01x03, J12 Conn_02x04_Odd_Even, J13 Screw_Terminal_01x03, J14 Screw_Terminal_01x03, J15 Screw_Terminal_01x03, J16 Screw_Terminal_01x03, J17 Screw_Terminal_01x03, J2 Screw_Terminal_01x03, J3 Screw_Terminal_01x03, J4 Screw_Terminal_01x03, J5 Screw_Terminal_01x03, J6 Screw_Terminal_01x03, J7 Screw_Terminal_01x03, J8 Screw_Terminal_01x03, J9 Screw_Terminal_01x03, K1 HF46F, K10 HF46F, K11 HF46F, K12 HF46F, K13 HF46F, K14 HF46F, K15 HF46F, K16 HF46F, K17 HF46F, K18 HF46F, K19 HF46F, K2 HF46F, K20 HF46F, K21 HF46F, K22 HF46F, K23 HF46F, K24 HF46F, K25 HF46F, K26 HF46F, K27 HF46F, K28 HF46F, K29 HF46F, K3 HF46F, K30 HF46F, K31 HF46F, K32 HF46F, K4 HF46F, K5 HF46F, K6 HF46F, K7 HF46F, K8 HF46F, K9 HF46F, U1 MCP23017_SS, U2 ULN2803A, U3 ULN2803A, U4 MCP23017_SS, U5 ULN2803A, U6 ULN2803A, U7 MCP9808_SO8, U8 MCP9808_MSOP

Commit message: relay_board_32x5A_v0.4
v0.4
Parts:
- removed A0 (x3), A1 (x3), A2 (x3): NO_Small, Jumper:SolderJumper-2_P1.3mm_Open_RoundedPad1.0x1.5mm
- removed JP7: SolderJumper_3_Open, Jumper:SolderJumper-3_P1.3mm_Bridged12_RoundedPad1.0x1.5mm
- removed the R10 at (381.9, 300.9)
- removed the R9 at (383.9, 300.9)
- added D1: LL4148, Diode_SMD:D_MiniMELF, F.Cu at (296.8, 324.8)
- added D10: LL4148, Diode_SMD:D_MiniMELF, F.Cu at (404.5, 324.8)
- added D11: LL4148, Diode_SMD:D_MiniMELF, F.Cu at (416.6, 324.8)
- added D12: LL4148, Diode_SMD:D_MiniMELF, F.Cu at (428.6, 324.8)
- added D13: LL4148, Diode_SMD:D_MiniMELF, F.Cu at (440.5, 324.8)
- added D14: LL4148, Diode_SMD:D_MiniMELF, F.Cu at (452.3, 324.8)
- added D15: LL4148, Diode_SMD:D_MiniMELF, F.Cu at (464.5, 324.8)
- added D16: LL4148, Diode_SMD:D_MiniMELF, F.Cu at (476.6, 324.8)
- added D17: LL4148, Diode_SMD:D_MiniMELF, F.Cu at (296.6, 298.7)
- added D18: LL4148, Diode_SMD:D_MiniMELF, F.Cu at (308.6, 298.7)
- added D19: LL4148, Diode_SMD:D_MiniMELF, F.Cu at (320.7, 298.7)
- added D2: LL4148, Diode_SMD:D_MiniMELF, F.Cu at (308.7, 324.8)
- added D20: LL4148, Diode_SMD:D_MiniMELF, F.Cu at (332.6, 298.7)
- added D21: LL4148, Diode_SMD:D_MiniMELF, F.Cu at (344.7, 298.7)
- added D22: LL4148, Diode_SMD:D_MiniMELF, F.Cu at (356.6, 298.7)
- added D23: LL4148, Diode_SMD:D_MiniMELF, F.Cu at (368.5, 298.7)
- added D24: LL4148, Diode_SMD:D_MiniMELF, F.Cu at (380.6, 298.7)
- added D25: LL4148, Diode_SMD:D_MiniMELF, F.Cu at (392.7, 298.7)
- added D26: LL4148, Diode_SMD:D_MiniMELF, F.Cu at (404.5, 298.7)
- added D27: LL4148, Diode_SMD:D_MiniMELF, F.Cu at (416.4, 298.7)
- added D28: LL4148, Diode_SMD:D_MiniMELF, F.Cu at (428.5, 298.7)
- added D29: LL4148, Diode_SMD:D_MiniMELF, F.Cu at (440.5, 298.7)
- added D3: LL4148, Diode_SMD:D_MiniMELF, F.Cu at (320.7, 324.8)
- added D30: LL4148, Diode_SMD:D_MiniMELF, F.Cu at (452.6, 298.7)
- added D31: LL4148, Diode_SMD:D_MiniMELF, F.Cu at (464.6, 298.7)
- added D32: LL4148, Diode_SMD:D_MiniMELF, F.Cu at (476.7, 298.7)
- added D4: LL4148, Diode_SMD:D_MiniMELF, F.Cu at (332.6, 324.8)
- added D5: LL4148, Diode_SMD:D_MiniMELF, F.Cu at (344.6, 324.8)
- added D6: LL4148, Diode_SMD:D_MiniMELF, F.Cu at (356.5, 324.8)
- added D7: LL4148, Diode_SMD:D_MiniMELF, F.Cu at (368.6, 324.8)
- added D8: LL4148, Diode_SMD:D_MiniMELF, F.Cu at (380.6, 324.8)
- added D9: LL4148, Diode_SMD:D_MiniMELF, F.Cu at (392.5, 324.8)
- added JP1: SolderJumper_3_Open, Jumper:SolderJumper-3_P1.3mm_Bridged12_RoundedPad1.0x1.5mm, B.Cu at (379.4, 317.3)
- added SW1: SW_DIP_x03, Button_Switch_SMD:SW_DIP_SPSTx03_Slide_Omron_A6S-310x_W8.9mm_P2.54mm, F.Cu at (353.4, 315.9)
- added SW2: SW_DIP_x03, Button_Switch_SMD:SW_DIP_SPSTx03_Slide_Omron_A6S-310x_W8.9mm_P2.54mm, F.Cu at (430.8, 315.9)
- added SW3: SW_DIP_x03, Button_Switch_SMD:SW_DIP_SPSTx03_Slide_Omron_A6S-310x_W8.9mm_P2.54mm, F.Cu at (473.0, 310.3)
- U8: value MCP9808_MSOP -> LM75_MSOP
- moved C7 17.3 mm to (460.2, 309.5), turned to 0 degrees
- moved R12 16.5 mm to (460.3, 306.1)
- moved R13 16.1 mm to (460.3, 307.8), turned to 0 degrees
- moved C3 6.98 mm to (373.8, 307.1)
- moved U3 6.95 mm to (366.4, 311.6)
- moved C6 6.86 mm to (451.1, 307.1)
- moved U6 6.83 mm to (443.8, 311.6)
- moved U8 5.85 mm to (463.0, 314.0)
- moved U7 5.85 mm to (463.0, 313.8)
- moved R1 5.40 mm to (340.5, 319.0), turned to -90 degrees
- moved R5 3.90 mm to (418.1, 319.0), turned to -90 degrees
- moved C4 3.21 mm to (414.1, 315.7), turned to 90 degrees
- moved R8 3.05 mm to (421.8, 319.0), turned to -90 degrees
- moved C1 3.04 mm to (336.5, 315.7), turned to 90 degrees
- moved R3 2.88 mm to (342.3, 319.0), turned to -90 degrees
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- renumbered R12 to R10, R13 to R11, R14 to R12, R15 to R13, R11 to R9
Connections:
- U1 pad 11: Net-(U1-Pad11) -> unconnected-(U1-Pad11)
- U1 pad 14: Net-(U1-Pad14) -> unconnected-(U1-Pad14)
- U1 pad 19: Net-(U1-Pad19) -> unconnected-(U1-Pad19)
- U1 pad 20: Net-(U1-Pad20) -> unconnected-(U1-Pad20)
- U4 pad 11: Net-(U4-Pad11) -> unconnected-(U4-Pad11)
- U4 pad 14: Net-(U4-Pad14) -> unconnected-(U4-Pad14)
- U4 pad 19: Net-(U4-Pad19) -> unconnected-(U4-Pad19)
- U4 pad 20: Net-(U4-Pad20) -> unconnected-(U4-Pad20)
Routing:
- net VCC: track 629.0 -> 727.3 mm, vias 5 -> 4
- net +3V3: track 264.4 -> 244.4 mm, vias 5 -> 9
- net Net-(R13-Pad2): track 19.5 -> 4.79 mm, vias 2 -> 0
- net SCL: track 164.5 -> 152.0 mm
- net RELAY17: track 62.7 -> 74.1 mm
- net RELAY25: track 44.7 -> 55.0 mm
- net RELAY18: track 53.4 -> 63.7 mm
- net SDA: track 164.0 -> 154.1 mm, vias 4 -> 6
- net GND: track 6.88 -> 16.3 mm, vias 127 -> 146
- net RELAY21: track 22.1 -> 31.5 mm
- net RELAY19: track 43.6 -> 52.8 mm
- net RELAY27: track 24.7 -> 33.7 mm
- net RELAY28: track 14.0 -> 22.7 mm
- net RELAY20: track 32.9 -> 41.3 mm
- net Net-(U1-Pad28): track 21.5 -> 29.8 mm
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Other:
- outline, holes or cut-outs redrawn
- net class +5V removed
- net class 230v removed
- net class Default removed
- board text added: "A0"
- board text added: "A1"
- board text added: "A2"
- board text added: "Relay Board 32x5A v0.4"
- board text removed: "Relay Board 32x5A v0.3"
